Commit message: Corrections

File: src/my_robot/urdf/my_robot.xacro (robot description, xacro)
@@ -138,5 +138,5 @@
   </joint>
   <joint name="right_wheel_hinge" type="continuous">
-    <origin xyz="0 0.15 0" rpy="0 0 0" />
+    <origin xyz="0 -0.15 0" rpy="0 0 0" />
     <parent link="chassis" />
     <child link="right_wheel" />
@@ -146,5 +146,5 @@
   </joint>
   <joint name="left_wheel_hinge" type="continuous">
-    <origin xyz="0 -0.15 0" rpy="0 0 0" />
+    <origin xyz="0 0.15 0" rpy="0 0 0" />
     <parent link="chassis" />
     <child link="left_wheel" />

Commit message: Fixing map appearance in rviz

File: src/my_robot/urdf/my_robot.xacro (robot description, xacro)
@@ -133,5 +133,5 @@
 <!-- JOINTS -->
   <joint name="robot_footprint_joint" type="fixed">
-    <origin xyz="0 0 0" rpy="0 0 0" />
+    <origin xyz="0 0 0.1" rpy="0 0 0" />
     <parent link="robot_footprint"/>
     <child link="chassis" />
